Commit message: Change allegro urdf to https://github.com/simlabrobotics/allegro_hand_ros_v4/blob/master/src/allegro_hand_description/urdf/allegro_hand_description_right.urdf, but change palm_link to base_link

File: grasp_generation/allegro_hand_description/allegro_hand_description_right.urdf (robot description, URDF)
Before this commit: robot allegro_hand_right, 21 links, 20 joints
Links:
- link base_link: mass None -> 0.4154
- link link_0.0: mass None -> 0.0119
- link link_1.0: mass None -> 0.065
- link link_10.0: mass None -> 0.0355
- link link_11.0: mass None -> 0.0096
- link link_11.0_tip: mass None -> 0.0168
- link link_12.0: mass None -> 0.0176
- link link_13.0: mass None -> 0.0119
- link link_14.0: mass None -> 0.038
- link link_15.0: mass None -> 0.0388
- link link_15.0_tip: mass None -> 0.0168
- link link_2.0: mass None -> 0.0355
- link link_3.0: mass None -> 0.0096
- link link_3.0_tip: mass None -> 0.0168
- link link_4.0: mass None -> 0.0119
- link link_5.0: mass None -> 0.065
- link link_6.0: mass None -> 0.0355
- link link_7.0: mass None -> 0.0096
- link link_7.0_tip: mass None -> 0.0168
- link link_8.0: mass None -> 0.0119
- link link_9.0: mass None -> 0.065
Joints:
- joint joint_0.0: limit lower=-0.47 upper=0.47 effort=0 velocity=0 -> lower=-0.47 upper=0.47 effort=15 velocity=7
- joint joint_1.0: limit lower=-0.196 upper=1.61 effort=0 velocity=0 -> lower=-0.196 upper=1.61 effort=15 velocity=7
- joint joint_10.0: limit lower=-0.174 upper=1.709 effort=0 velocity=0 -> lower=-0.174 upper=1.709 effort=15 velocity=7
- joint joint_11.0: limit lower=-0.227 upper=1.618 effort=0 velocity=0 -> lower=-0.227 upper=1.618 effort=15 velocity=7
- joint joint_12.0: limit lower=0.263 upper=1.396 effort=0 velocity=0 -> lower=0.263 upper=1.396 effort=15 velocity=7
- joint joint_13.0: limit lower=-0.105 upper=1.163 effort=0 velocity=0 -> lower=-0.105 upper=1.163 effort=15 velocity=7
- joint joint_14.0: limit lower=-0.189 upper=1.644 effort=0 velocity=0 -> lower=-0.189 upper=1.644 effort=15 velocity=7
- joint joint_15.0: limit lower=-0.162 upper=1.719 effort=0 velocity=0 -> lower=-0.162 upper=1.719 effort=15 velocity=7
- joint joint_2.0: limit lower=-0.174 upper=1.709 effort=0 velocity=0 -> lower=-0.174 upper=1.709 effort=15 velocity=7
- joint joint_3.0: limit lower=-0.227 upper=1.618 effort=0 velocity=0 -> lower=-0.227 upper=1.618 effort=15 velocity=7
- joint joint_4.0: limit lower=-0.47 upper=0.47 effort=0 velocity=0 -> lower=-0.47 upper=0.47 effort=15 velocity=7
- joint joint_5.0: limit lower=-0.196 upper=1.61 effort=0 velocity=0 -> lower=-0.196 upper=1.61 effort=15 velocity=7
- joint joint_6.0: limit lower=-0.174 upper=1.709 effort=0 velocity=0 -> lower=-0.174 upper=1.709 effort=15 velocity=7
- joint joint_7.0: limit lower=-0.227 upper=1.618 effort=0 velocity=0 -> lower=-0.227 upper=1.618 effort=15 velocity=7
- joint joint_8.0: limit lower=-0.47 upper=0.47 effort=0 velocity=0 -> lower=-0.47 upper=0.47 effort=15 velocity=7
- joint joint_9.0: limit lower=-0.196 upper=1.61 effort=0 velocity=0 -> lower=-0.196 upper=1.61 effort=15 velocity=7
